File: WROVER-Nextion3.5/ClimateSprinklerController.sch (KiCad schematic (older format))
At the start: 113 parts, among them J1 USB_B_Micro, J2 7.5 TO 40 V, J3 NEXTION, J4 SERIAL, J5 SPI, J6 PIR, J7 I2C, Q1 MMSS8050, Q2 MMSS8050, Q3 TEPT5700, SW1 POWER, SW2 RESET, SW3 MODE, U1 ESP32-WROVER, U10 BME280, U11 DHT22, U2 FT232RL, U3 LMR36520, U4 TPS22917DBV, U5 SGP40-Sensor_Air_Quality, U6 LD1086DT33TR, U7 SHTC3, U8 BME680, U9 TMP117

Commit message: Nextion PCBs tweak
Parts:
- J2: value 7.5 TO 40 V -> 5 TO 40 V*
Changed lines of the file:
@@
 P 1425 1500
 F 0 "J2" H 1195 1542 50  0000 R CNN
-F 1 "7.5 TO 40 V" H 1195 1451 50  0000 R CNN
+F 1 "5 TO 40 V*" H 1195 1451 50  0000 R CNN
 F 2 "Connector_BarrelJack:BarrelJack_Horizontal" H 1475 1460 50  0001 C CNN
 F 3 "~" H 1475 1460 50  0001 C CNN

Commit message: TX+RX LEDs were backwards...oops
Connections:
- net at C10.1, R5.1, U2.17 (3V3OUT)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: now also D3.2 (A), D4.2 (A); no longer D3.1 (K), D4.1 (K)
- net at R3.1: now also D3.1 (K); no longer D3.2 (A)
- net at R4.1: now also D4.1 (K); no longer D4.2 (A)
Other:
- moved on the sheet: D3, D4
Changed lines of the file:
@@
 F 4 "APTL3216QBC/D" V 4925 8700 50  0001 C CNN "Part"
 	1    4925 8700
-	-1   0    0    1
+	1    0    0    1
 $EndComp
 $Comp
@@
 F 4 "APTL3216SURCK" V 4925 9000 50  0001 C CNN "Part"
 	1    4925 9000
-	-1   0    0    1
+	1    0    0    1
 $EndComp
 Wire Wire Line

Commit message: Doc updates, new images, new enclosures, regenerate gerbers
Parts:
- C1, C13, C6, C7: MPN1 (none) -> C2012X5R1H475K125AB; Part C2012X5R1H475K125AB -> (none)
- C10, C11, C15, C17, C19, C2, C23, C24, C25, C26, C27, C28, C29, C30, C31, C4: MPN1 (none) -> CC0805KRX7R7BB104; Part CC0805KRX7R7BB104 -> (none)
- C12, C14, C16: MPN1 (none) -> GRM32ER61C476KE15L; Part GRM32ER61C476KE15L -> (none)
- C18, C22: MPN1 (none) -> EEE-HP0J100R; Part EEE-HP0J100R -> (none)
- C20, C21, C9: MPN1 (none) -> C0805C105K4RACTU; Part C0805C105K4RACTU -> (none)
- C3: MPN1 (none) -> C2012X5R1V106K085AC; Part C2012X5R1V106K085AC -> (none)
- C5: MPN1 (none) -> 25SVF100M; Part 25SVF100M -> (none)
- C8: MPN1 (none) -> C2012X5R1H224K125AA; Part C2012X5R1H224K125AA -> (none)
- D1, D2: value MBR230S1F-7 -> N/A; MPN1 (none) -> MBR230S1F-7; Part MBR230S1F-7 -> (none)
- D3: MPN1 (none) -> APTL3216QBC/D; Part APTL3216QBC/D -> (none)
- D4: MPN1 (none) -> APTL3216SURCK; Part APTL3216SURCK -> (none)
- D5: MPN1 (none) -> APTL3216ZGC; Part APTL3216ZGC -> (none)
- D6, D7: MPN1 (none) -> 597-6901-607F; Part 597-6901-607F -> (none)
- D8: MPN1 (none) -> APTL3216SECK; Part APTL3216SECK -> (none)
- F1: MPN1 (none) -> 2920L075; Part 2920L075 -> (none)
- H1, H2, H3, H4, H5, H6, H7, H8, J3, J4, J5, J6, J7, JP1, JP10, JP11, JP12, JP2, JP3, JP4, JP5, JP6, JP7, JP8, JP9: MPN1 (none) -> N/A; Population (none) -> DNF
- J1: value USB_B_Micro -> N/A; MPN1 (none) -> 105017-0001; Part 105017-0001 -> (none)
- J2: MPN1 (none) -> 694106301002; Part 694106301002 -> (none)
- L1: MPN1 (none) -> 7447709150; MPN2 (none) -> MSS1210-153MEB; Part 7447709150 -> (none); PartAlt MSS1210-153MEB -> (none)
- Q1, Q2: MPN1 (none) -> MMSS8050; Part MMSS8050 -> (none)
- Q3: MPN1 (none) -> TEPT5700; Part TEPT5700 -> (none)
- R1: MPN1 (none) -> RT0805FRE074K7L; Part RT0805FRE074K7L -> (none)
- R10: MPN1 (none) -> RT0805FRE0724K9L; Part RT0805FRE0724K9L -> (none)
- R11, R12, R13, R14, R15, R2, R22, R24, R25, R26, R5: MPN1 (none) -> RC0805FR-0710KL; Part RC0805FR-0710KL -> (none)
- R16: MPN1 (none) -> RT0805FRE078K2L; Part RT0805FRE078K2L -> (none)
- R17, R18: MPN1 (none) -> RC0805FR-074R7L; Part RC0805FR-074R7L -> (none)
- R19: MPN1 (none) -> RT0805FRE071K6L; Part RT0805FRE071K6L -> (none)
- R20, R9: MPN1 (none) -> RC0805FR-07100KL; Part RC0805FR-07100KL -> (none)
- R21: MPN1 (none) -> RT0805FRE07120RL; Part RT0805FRE07120RL -> (none)
- R23: MPN1 (none) -> CRCW08055K00JNTA; Part CRCW08055K00JNTA -> (none)
- R3, R4: MPN1 (none) -> RT0805FRE072K7L; Part RT0805FRE072K7L -> (none)
- R6, R8: MPN1 (none) -> RT0805FRE073K3L; Part RT0805FRE073K3L -> (none)
- R7: MPN1 (none) -> RC0805FR-0710KL; Part RT0805FRE079K1L -> (none)
- SW1: MPN1 (none) -> 48BFSP1M6QT; Part 48BFSP1M6QT -> (none)
- SW2, SW3: MPN1 (none) -> PTS645VK582LFS; Part PTS645VK582LFS -> (none)
- TH1, TH2: value NXFT15XH103FA2B100 -> 10K; MPN1 (none) -> NXFT15XH103FA2B100; Part NXFT15XH103FA2B100 -> (none)
- U1: MPN1 (none) -> ESP32-WROVER; Part ESP32-WROVER -> (none)
- U10: MPN1 (none) -> BME280; Part BME280 -> (none)
- U11: MPN1 (none) -> DHT22; Part DHT22 -> (none)
- U2: MPN1 (none) -> FT232RL; Part FT232RL -> (none)
- U3: MPN1 (none) -> LMR36520ADDAR; Part LMR36520ADDAR -> (none)
- U4: MPN1 (none) -> TPS22917DBV; Part TPS22917DBV -> (none)
- U5: value SGP40-Sensor_Air_Quality -> SGP40; MPN1 (none) -> SGP40; Part SGP40 -> (none)
- U6: MPN1 (none) -> LD1086DT33TR; Part LD1086DT33TR -> (none)
- U7: MPN1 (none) -> SHTC3; Part SHTC3 -> (none)
- U8: MPN1 (none) -> BME680; Part BME680 -> (none)
- U9: MPN1 (none) -> TMP117MAIDRVR; Part TMP117MAIDRVR -> (none)
Connections:
- net +3V3: now also C31.1, U11.1 (VCC)
- net +5V: no longer C31.1, U11.1 (VCC)
