File: WROVER-Nextion7/ClimateSprinklerController.kicad_pcb (KiCad board)
At the start: 2 copper layers, 217 x 108 mm, 227 parts, among them J1 7.5 TO 40 V, J10 HVAC, J11 RELAY, J2 USB_B_Micro, J3 POWER SEL, J4 NEXTION, J5 SERIAL, J6 SPI, J7 PIR, J8 I2C, J9 IO_EXP, K1 G6E-134P-US DC5, K2 G6E-134P-US DC5, K3 G6E-134P-US DC5, Q1 MMSS8050, Q10 2N6073B, Q11 2N6073B, Q12 2N6073B, Q13 2N6073B, Q14 2N6073B, Q2 MMSS8050, Q3 TEPT5700, Q4 2N7002, Q5 2N7002, Q6 2N7002, Q7 2N6073B, Q8 2N6073B, Q9 2N6073B, SW1 POWER, SW2 RESET, SW3 MODE, U1 ESP32-WROVER, U10 SHTC3, U11 TMP117, U12 MOC3043, U13 MOC3043, U14 MOC3043, U15 MOC3043, U16 MOC3043, U17 MOC3043, U18 MOC3043, U19 MOC3043, U2 MCP23017_SO, U20 DHT22, U3 FT232RL, U4 TPS22917DBV, U5 LMR36520, U6 SGP40-Sensor_Air_Quality, U7 BME680, U8 LD1086DT33TR, U9 BME280

Commit message: TX+RX LEDs were backwards...oops
Connections:
- D3 pad 1: Net-(C11-Pad1) -> Net-(D3-Pad1)
- D3 pad 2: Net-(D3-Pad2) -> Net-(C11-Pad1)
- D4 pad 1: Net-(C11-Pad1) -> Net-(D4-Pad1)
- D4 pad 2: Net-(D4-Pad2) -> Net-(C11-Pad1)
- R10 pad 1: Net-(D4-Pad2) -> Net-(D4-Pad1)
- R9 pad 1: Net-(D3-Pad2) -> Net-(D3-Pad1)
Routing:
- net Net-(D4-Pad2): track 7.76 -> 0.00 mm
- net Net-(D3-Pad2): track 7.76 -> 0.00 mm
- net Net-(C11-Pad1): track 38.9 -> 42.2 mm
- net Net-(D4-Pad1): track 0.00 -> 2.70 mm
- net Net-(D3-Pad1): track 0.00 -> 2.70 mm

Commit message: Doc updates, new images, new enclosures, regenerate gerbers
Parts:
- C32: moved to F.Cu
- D1: value MBR230S1F-7 -> N/A
- D11, D13, D9: value 1N4148 -> N/A
- D2: value CD-MBL206SL -> N/A
- J2: value USB_B_Micro -> N/A
- R29, R30, R31: value 1K2 -> 560
- R33, R34, R37, R38, R39: value 1K2 -> 1K5
- RV1: value B72205S0400K101 -> N/A
- TH1: value NXFT15XH103FA2B100 -> 10K
- U11: value TMP117 -> TMP117MAIDRVR
- U12, U13, U14, U15, U16, U17, U18, U19: value MOC3043 -> MOC3043SM
- U2: value MCP23017_SO -> MCP23017-E/SO
- U5: value LMR36520 -> LMR36520ADDAR
- U6: value SGP40-Sensor_Air_Quality -> SGP40
Connections:
- C32 pad 1: +5V -> +3V3
- U20 pad 1: +5V -> +3V3
Routing:
- net +5V: track 402.5 -> 357.0 mm
- net +3V3: track 431.4 -> 445.1 mm
